File: MD02F-2 MGD2 Mainboard/MD02F-2.kicad_pcb (KiCad board)
At the start: 2 copper layers, 107.1 x 135.2 mm, 76 parts, among them CON1 Adapter Connector, CON2 Floppy Disk Drive Connector, CON3 Conn_01x02, CON4 Power Connector, SW1 Select, SW2 Minus, SW3 Plus, U7 74LS244

Commit message: Add files via upload
Connections:
- net /CON1.Pin2 renamed /CON1.A16
- net /CON1.Pin3 renamed /CON1.A15
- net /CON1.Pin37 renamed /~{Read}.RAM8
- net /CON1.Pin38 renamed /~{Read}.RAM5
- net /CON1.Pin39 renamed /~{Read}.RAM7
- net /CON1.Pin40 renamed /~{Read}.RAM6
- net /CON1.Pin41 renamed /~{Read}.RAM1
- net /CON1.Pin42 renamed /~{Read}.RAM4
- net /CON1.Pin43 renamed /~{Read}.RAM2
- net /CON1.Pin44 renamed /~{Read}.RAM3
- net /CON1.Pin45 renamed /Batt.Detect
- net /CON1.Pin50 renamed /74HC161D.CP
- CON1 pad 47: unconnected-(CON1-Pin_47-Pad47) -> /Counter.Bit2
- CON1 pad 48: unconnected-(CON1-Pin_48-Pad48) -> /Counter.Bit1
- CON1 pad 49: unconnected-(CON1-Pin_49-Pad49) -> /Counter.Bit0
