File: MD02F-2 MGD2 Mainboard/MD02F-2.kicad_sch (KiCad schematic)
At the start: 76 parts, among them CON1 Adapter Connector, CON2 Floppy Disk Drive Connector, CON3 Conn_01x02, CON4 Power Connector, SW1 Select, SW2 Minus, SW3 Plus, U7 74LS244

Commit message: Add files via upload
Connections:
- net Counter.Bit2: now reaches CON1.47 (Pin_47)
- net Counter.Bit1: now reaches CON1.48 (Pin_48)
- net Counter.Bit0: now reaches CON1.49 (Pin_49)
- net CON1.Pin2 renamed CON1.A16
- net CON1.Pin3 renamed CON1.A15
- net CON1.Pin37 renamed ~{Read}.RAM8
- net CON1.Pin38 renamed ~{Read}.RAM5
- net CON1.Pin39 renamed ~{Read}.RAM7
- net CON1.Pin40 renamed ~{Read}.RAM6
- net CON1.Pin41 renamed ~{Read}.RAM1
- net CON1.Pin42 renamed ~{Read}.RAM4
- net CON1.Pin43 renamed ~{Read}.RAM2
- net CON1.Pin44 renamed ~{Read}.RAM3
- net CON1.Pin45 renamed Batt.Detect
- net CON1.Pin50 renamed 74HC161D.CP
- no-connect marks 27 -> 24
