File: MD02U-1 Cartridge Adapter Board/MD02U-1.kicad_pcb (KiCad board)
At the start: 2 copper layers, 152.4 x 165 mm, 22 parts, among them CON1 MGD2 Edge Connector, CON2 Conn_01x06_Pin, J1 GG Cartridge Slot, J2 GB Cartridge Slot, J3 SNES Cartridge Slot, J4 Sega MegaDrive Cartridge Slot, J5 PCE Cartridge Slot, U1 74LS245 - BUSA, U2 74LS245 - BUSB, U3 74LS273 - BANK, U4 PEEL

Commit message: Add files via upload
Routing:
- net /D1.Carts: track 285.4 -> 288.4 mm
- net /D3.Carts: track 288.1 -> 291.2 mm
- net /D6.Carts: track 254.7 -> 257.6 mm
- net /~{Read}: track 347.3 -> 350.3 mm

Commit message: Add files via upload
Parts:
- U4: value PEEL -> ~
Connections:
- net /CON1.Pin38 renamed /~{Read}.U5
- net /CON1.Pin39 renamed /~{Read}.U7
- net /CON1.Pin40 renamed /~{Read}.U6
- net /CON1.Pin42 renamed /~{Read}.U4
- net /CON1.Pin45 renamed /Batt.Detect
- net /~{Read} renamed /~{Read}.U8
