File: MD02U-1 Cartridge Adapter Board/MD02U-1.kicad_sch (KiCad schematic)
At the start: 22 parts, among them CON1 MGD2 Edge Connector, CON2 Conn_01x06_Pin, J1 GG Cartridge Slot, J2 GB Cartridge Slot, J3 SNES Cartridge Slot, J4 Sega MegaDrive Cartridge Slot, J5 PCE Cartridge Slot, U1 74LS245 - BUSA, U2 74LS245 - BUSB, U3 74LS273 - BANK

Commit message: Add files via upload
Connections:
- net CON1.Pin38 renamed ~{Read}.U5
- net CON1.Pin39 renamed ~{Read}.U7
- net CON1.Pin40 renamed ~{Read}.U6
- net CON1.Pin42 renamed ~{Read}.U4
- net CON1.Pin45 renamed Batt.Detect
- net ~{Read} renamed ~{Read}.U8
Changed lines of the file:
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@@
 (kicad_sch
-	(version 20231120)
+	(version 20250114)
 	(generator "eeschema")
-	(generator_version "8.0")
+	(generator_version "9.0")
 	(paper "A3")
 	(junction
@@
 		)
 	)
-	(label "CON1.Pin38"
+	(label "~{Read}.U5"
 		(at 80.01 248.92 270)
 		(effects
@@
 		)
 	)
-	(label "CON1.Pin42"
+	(label "~{Read}.U4"
 		(at 326.39 176.53 180)
 		(effects
@@
 		)
 	)
+	(label "~{Read}.U8"
+		(at 326.39 173.99 180)
+		(effects
+			(font
+				(size 1.27 1.27)
+			)
+			(justify right bottom)
+		)
+	)
 	(label "D3.MGD2"
 		(at 227.33 173.99 0)
@@
 		)
 	)
-	(label "CON1.Pin45"
+	(label "Batt.Detect"
 		(at 232.41 260.35 270)
 		(effects
@@
 		)
 	)
-	(label "CON1.Pin42"
+	(label "~{Read}.U4"
 		(at 227.33 247.65 90)
 		(effects
@@
 		)
 	)
-	(label "~{Read}"
-		(at 232.41 80.01 0)
-		(effects
-			(font
-				(size 1.27 1.27)
-			)
-			(justify left bottom)
-		)
-	)
 	(label "GG.GB.~{Read}"
 		(at 356.87 173.99 0)
@@
 		)
 	)
-	(label "CON1.Pin39"
+	(label "~{Read}.U7"
 		(at 224.79 260.35 270)
 		(effects
@@
 		)
 	)
-	(label "~{Read}"
-		(at 359.41 73.66 0)
-		(effects
-			(font
-				(size 1.27 1.27)
-			)
-			(justify left bottom)
-		)
-	)
 	(label "A10"
 		(at 138.43 80.01 180)
@@
 		)
 	)
-	(label "~{Read}"
+	(label "~{Read}.U8"
 		(at 222.25 260.35 270)
 		(effects
@@
 		)
 	)
-	(label "~{Read}"
-		(at 200.66 92.71 180)
-		(effects
-			(font
-				(size 1.27 1.27)
-			)
-			(justify right bottom)
-		)
-	)
 	(label "A7"
 		(at 138.43 72.39 180)
@@
 		)
 	)
-	(label "CON1.Pin40"
+	(label "~{Read}.U6"
 		(at 105.41 241.3 0)
 		(effects
@@
 		)
 	)
+	(label "~{Read}.U8"
+		(at 232.41 80.01 0)
+		(effects
+			(font
+				(size 1.27 1.27)
+			)
+			(justify left bottom)
+		)
+	)
 	(label "A3"
 		(at 138.43 62.23 180)
@@
 		)
 	)
-	(label "CON1.Pin45"
+	(label "Batt.Detect"
 		(at 57.15 246.38 0)
 		(effects
@@
 		)
 	)
+	(label "~{Read}.U8"
+		(at 261.62 73.66 180)
+		(effects
+			(font
+				(size 1.27 1.27)
+			)
+			(justify right bottom)
+		)
+	)
 	(label "A16"
 		(at 284.48 168.91 0)
@@
 		)
 	)
-	(label "~{Read}"
+	(label "~{Read}.U8"
 		(at 97.79 60.96 0)
 		(effects
@@
 		)
 	)
+	(label "~{Read}.U8"
+		(at 261.62 76.2 180)
+		(effects
+			(font
+				(size 1.27 1.27)
+			)
+			(justify right bottom)
+		)
+	)
 	(label "+5V"
 		(at 232.41 102.87 0)
@@
 		)
 	)
-	(label "~{Read}"
-		(at 261.62 76.2 180)
-		(effects
-			(font
-				(size 1.27 1.27)
-			)
-			(justify right bottom)
-		)
-	)
 	(label "D2.Carts"
 		(at 71.12 194.31 270)
@@
 		)
 	)
-	(label "~{Read}"
-		(at 326.39 173.99 180)
-		(effects
-			(font
-				(size 1.27 1.27)
-			)
-			(justify right bottom)
-		)
-	)
 	(label "D12.MD"
 		(at 261.62 96.52 180)
@@
 		)
 	)
-	(label "~{Read}"
-		(at 261.62 73.66 180)
-		(effects
-			(font
-				(size 1.27 1.27)
-			)
-			(justify right bottom)
-		)
-	)
 	(label "A9"
 		(at 97.79 68.58 0)
@@
 		)
 	)
-	(label "CON1.Pin40"
+	(label "~{Read}.U6"
 		(at 224.79 247.65 90)
 		(effects
@@
 		)
 	)
-	(label "CON1.Pin39"
+	(label "~{Read}.U7"
 		(at 80.01 233.68 90)
 		(effects
@@
 		)
 	)
+	(label "~{Read}.U8"
+		(at 359.41 73.66 0)
+		(effects
+			(font
+				(size 1.27 1.27)
+			)
+			(justify left bottom)
+		)
+	)
 	(label "GND"
 		(at 59.69 82.55 180)
@@
 		)
 	)
+	(label "~{Read}.U8"
+		(at 200.66 92.71 180)
+		(effects
+			(font
+				(size 1.27 1.27)
+			)
+			(justify right bottom)
+		)
+	)
 	(label "A6"
 		(at 189.23 247.65 90)
@@
 		)
 	)
-	(label "CON1.Pin38"
+	(label "~{Read}.U5"
 		(at 222.25 247.65 90)
 		(effects
@@
 		)
 	)
+	(embedded_fonts no)
 )
